File: hardware/nfc_copy_cat.sch (KiCad schematic (older format))
At the start: 36 parts, among them J1 USB_B_Micro, J2 Battery, J3 SWD, J4 NFC Module V3, J5 Conn_01x02, J6 Adafruit NFC 1.0, SW1 RST, SW2 Magspoof, SW3 NFC, U1 AP2112K-3.3TRG1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

Commit message: fix caps, change SPI flash and LEDs, add ON/OFF
Parts:
- removed D1: POWER, LED_SMD:LED_0805_2012Metric_Pad1.15x1.40mm_HandSolder, symbol Device:LED_Small
- removed R1: 330, Resistor_SMD:R_0805_2012Metric_Pad1.15x1.40mm_HandSolder, symbol Device:R_Small
- added SW?: ON/OFF, symbol nfc_copy_cat-rescue:SW_DPST_x2-Switch
- C1: value 0.1uf -> 1uf
- C4: value 0.1uf -> 10uf
- J1: symbol Connector:USB_B_Micro -> nfc_copy_cat-rescue:USB_B_Micro-Connector
- R7: value 100K -> 10K
- U5: value W25Q16JVSS -> GD25Q16C
Connections:
- net labels added: MISO1, MOSI1, SCK1, SS1
- net labels removed: MISO, MOSI, SCK, SS
- wire segments 105 -> 115
Other:
- moved on the sheet: C8, D2, SW1A
