File: hardware/nfc_copy_cat.kicad_pcb (KiCad board)
At the start: 2 copper layers, 40.4 x 43 mm, 41 parts, among them J1 USB_B_Micro, J2 Battery, J3 SWD, J4 NFC Module V3, J5 Conn_01x02, J6 Adafruit NFC 1.0, SW1 RST, SW2 Magspoof, SW3 NFC, U1 AP2112K-3.3TRG1, U2 MCP73831-2-OT, U3 TC4424, U4 ATSAMD21E18A, U5 W25Q16JVSS

Commit message: change routeo
Parts:
- moved C2 3.51 mm to (152.2, 86.2), turned to 180 degrees
- moved U3 3.44 mm to (157.9, 89.2)
- moved J5 2.07 mm to (163.9, 87.5)
- moved D4 0.69 mm to (146.8, 70.2)
- moved C1 0.69 mm to (152.2, 84.2), turned to 180 degrees
- moved R4 0.67 mm to (144.3, 70.2)
Routing:
- net /SWDIO: track 0.00 -> 41.0 mm, vias 0 -> 1
- net GND: track 64.9 -> 102.9 mm, vias 6 -> 12
- net /SWCLK: track 0.00 -> 34.3 mm, vias 0 -> 1
- net /IN_A: track 0.00 -> 18.7 mm, vias 0 -> 2
- net /SS: track 9.06 -> 24.4 mm, vias 0 -> 2
- net +3V3: track 127.2 -> 142.4 mm, vias 1 -> 3
- net VCC: track 36.3 -> 44.9 mm
- net Net-(D6-Pad1): track 0.00 -> 5.30 mm, vias 0 -> 1
- net Net-(D5-Pad1): track 2.54 -> 5.23 mm
- net Net-(D4-Pad1): track 2.56 -> 5.08 mm
- net Net-(C1-Pad1): track 2.23 -> 4.17 mm
- net /IN_B: track 27.8 -> 26.4 mm, vias 2 -> 4
- net /11(MOSI): track 39.4 -> 40.6 mm, vias 4 -> 2
- net /OUTB: track 4.88 -> 3.90 mm
- net /OUTA: track 4.88 -> 3.90 mm
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
Commit message: fix c5 and sc
Parts:
- moved C5 1.08 mm to (138.3, 67.9), turned to 0 degrees
Routing:
- net /SS: track 24.4 -> 26.9 mm
- net +3V3: track 142.4 -> 141.6 mm
- net VCC: track 44.9 -> 44.1 mm
Changed lines of the file:
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@@
     (thickness 1.6)
     (drawings 32)
-    (tracks 574)
+    (tracks 566)
     (zones 0)
     (modules 41)
@@
   )
   (module Capacitor_SMD:C_0805_2012Metric_Pad1.15x1.40mm_HandSolder (layer F.Cu)
-    (at 137.23 67.775 270)
+    (at 138.31 67.865)
     (descr "Capacitor SMD 0805 (2012 Metric), square (rectangular) end terminal, IPC_7351 nominal with elongated pad for handsoldering. (Body size source: https://docs.google.com/spreadsheets/d/1BsfQQcO9C6DZCsRaXUlFlo91Tg2WpOkGARC1WS5S8t0/edit?usp=sharing), generated with kicad-footprint-generator")
     (tags "capacitor handsolder")
     (attr smd)
-    (fp_text reference C5 (at 2.8358 -0.1524 90) (layer F.SilkS)
+    (fp_text reference C5 (at 2.8358 -0.1524) (layer F.SilkS)
       (effects (font (size 1 1) (thickness 0.15)))
     )
-    (fp_text value 1uf (at 0 1.65 90) (layer F.Fab)
+    (fp_text value 1uf (at 0 1.65) (layer F.Fab)
       (effects (font (size 1 1) (thickness 0.15)))
     )
@@
     (fp_line (start 1.85 -0.95) (end 1.85 0.95) (layer F.CrtYd) (width 0.05))
     (fp_line (start 1.85 0.95) (end -1.85 0.95) (layer F.CrtYd) (width 0.05))
-    (fp_text user %R (at 0 0 90) (layer F.Fab)
+    (fp_text user %R (at 0 0) (layer F.Fab)
       (effects (font (size 0.5 0.5) (thickness 0.08)))
     )
-    (pad 1 smd roundrect (at -1.025 0 270) (size 1.15 1.4) (layers F.Cu F.Paste F.Mask) (roundrect_rratio 0.217391)
+    (pad 1 smd roundrect (at -1.025 0) (size 1.15 1.4) (layers F.Cu F.Paste F.Mask) (roundrect_rratio 0.217391)
       (net 3 VCC))
-    (pad 2 smd roundrect (at 1.025 0 270) (size 1.15 1.4) (layers F.Cu F.Paste F.Mask) (roundrect_rratio 0.217391)
+    (pad 2 smd roundrect (at 1.025 0) (size 1.15 1.4) (layers F.Cu F.Paste F.Mask) (roundrect_rratio 0.217391)
       (net 2 GND))
     (model ${KISYS3DMOD}/Capacitor_SMD.3dshapes/C_0805_2012Metric.wrl
@@
   (segment (start 141.2582 65.6082) (end 141.23 65.58) (width 0.5) (layer F.Cu) (net 1))
   (segment (start 147.022 65.6082) (end 141.2582 65.6082) (width 0.5) (layer F.Cu) (net 1))
-  (segment (start 138.4628 65.5768) (end 138.4396 65.6) (width 0.5) (layer F.Cu) (net 1))
-  (segment (start 139.2628 65.5768) (end 138.4628 65.5768) (width 0.5) (layer F.Cu) (net 1))
   (segment (start 132.6032 61.7336) (end 132.6 61.7304) (width 0.5) (layer F.Cu) (net 1))
   (segment (start 132.6032 63.0136) (end 132.6032 61.7336) (width 0.5) (layer F.Cu) (net 1))
@@
   (segment (start 130.9464 65.7136) (end 132.6032 65.7136) (width 0.5) (layer F.Cu) (net 3))
   (segment (start 130.5 66.16) (end 130.9464 65.7136) (width 0.5) (layer F.Cu) (net 3))
-  (segment (start 146.77 58.78) (end 146.77 59.8) (width 0.5) (layer F.Cu) (net 3))
-  (segment (start 146.77 59.8) (end 144.48 62.09) (width 0.5) (layer F.Cu) (net 3))
-  (segment (start 144.48 62.09) (end 137.73 62.09) (width 0.5) (layer F.Cu) (net 3))
   (via (at 137.73 62.09) (size 0.8) (drill 0.4) (layers F.Cu B.Cu) (net 3))
   (via (at 137.28 64.9) (size 0.8) (drill 0.4) (layers F.Cu B.Cu) (net 3))
   (segment (start 137.73 64.45) (end 137.28 64.9) (width 0.5) (layer B.Cu) (net 3))
   (segment (start 137.73 62.09) (end 137.73 64.45) (width 0.5) (layer B.Cu) (net 3))
-  (segment (start 137.28 66.7) (end 137.23 66.75) (width 0.5) (layer F.Cu) (net 3))
-  (segment (start 137.28 64.9) (end 137.28 66.7) (width 0.5) (layer F.Cu) (net 3))
-  (segment (start 135.87 73.27) (end 135.87 67.26) (width 0.5) (layer F.Cu) (net 3))
-  (segment (start 136.38 66.75) (end 137.23 66.75) (width 0.5) (layer F.Cu) (net 3))
-  (segment (start 135.87 67.26) (end 136.38 66.75) (width 0.5) (layer F.Cu) (net 3))
-  (segment (start 137.23 66.75) (end 136.29 66.75) (width 0.5) (layer F.Cu) (net 3))
-  (segment (start 134.7068 65.51) (end 134.5032 65.7136) (width 0.5) (layer F.Cu) (net 3))
-  (segment (start 135.05 65.51) (end 134.7068 65.51) (width 0.5) (layer F.Cu) (net 3))
-  (segment (start 135.87 67.26) (end 135.87 66.47) (width 0.5) (layer F.Cu) (net 3))
-  (segment (start 135.87 66.47) (end 135.94 66.4) (width 0.5) (layer F.Cu) (net 3))
-  (segment (start 135.94 66.4) (end 135.05 65.51) (width 0.5) (layer F.Cu) (net 3))
-  (segment (start 136.29 66.75) (end 135.94 66.4) (width 0.5) (layer F.Cu) (net 3))
+  (segment (start 137.285 64.905) (end 137.28 64.9) (width 0.5) (layer F.Cu) (net 3))
+  (segment (start 137.1436 65.7136) (end 137.285 65.855) (width 0.5) (layer F.Cu) (net 3))
+  (segment (start 136.7936 65.6164) (end 137.285 65.125) (width 0.5) (layer F.Cu) (net 3))
+  (segment (start 136.7936 65.7136) (end 136.7936 65.6164) (width 0.5) (layer F.Cu) (net 3))
+  (segment (start 137.285 65.855) (end 137.285 65.125) (width 0.5) (layer F.Cu) (net 3))
+  (segment (start 137.285 65.125) (end 137.285 64.905) (width 0.5) (layer F.Cu) (net 3))
+  (segment (start 134.5032 65.7136) (end 136.7936 65.7136) (width 0.5) (layer F.Cu) (net 3))
+  (segment (start 136.7936 65.7136) (end 137.1436 65.7136) (width 0.5) (layer F.Cu) (net 3))
+  (segment (start 137.285 66.205) (end 136.7936 65.7136) (width 0.5) (layer F.Cu) (net 3))
+  (segment (start 137.285 67.865) (end 137.285 66.325) (width 0.5) (layer F.Cu) (net 3))
+  (segment (start 137.285 66.325) (end 137.285 66.205) (width 0.5) (layer F.Cu) (net 3))
+  (segment (start 137.285 66.325) (end 137.285 65.855) (width 0.5) (layer F.Cu) (net 3))
+  (segment (start 143.46 62.09) (end 138.295685 62.09) (width 0.5) (layer F.Cu) (net 3))
+  (segment (start 146.77 58.78) (end 143.46 62.09) (width 0.5) (layer F.Cu) (net 3))
+  (segment (start 138.295685 62.09) (end 137.73 62.09) (width 0.5) (layer F.Cu) (net 3))
+  (segment (start 138.8285 73.2935) (end 138.8285 71.4285) (width 0.5) (layer F.Cu) (net 3))
+  (segment (start 137.285 69.885) (end 137.285 67.865) (width 0.5) (layer F.Cu) (net 3))
+  (segment (start 138.8285 71.4285) (end 137.285 69.885) (width 0.5) (layer F.Cu) (net 3))
   (segment (start 133.07 56.72) (end 133.03 56.76) (width 0.3) (layer F.Cu) (net 4))
   (segment (start 137.52 56.72) (end 133.07 56.72) (width 0.3) (layer F.Cu) (net 4))
@@
   (segment (start 158.95 61.85) (end 158.93 61.87) (width 0.3) (layer B.Cu) (net 43))
   (segment (start 158.95 60.08) (end 158.95 61.85) (width 0.3) (layer B.Cu) (net 43))
-  (segment (start 147.89 59.7274) (end 151.202 56.4154) (width 0.3) (layer F.Cu) (net 45))
-  (segment (start 147.89 60.98) (end 147.89 59.7274) (width 0.3) (layer F.Cu) (net 45))
-  (segment (start 151.202 56.4154) (end 151.877 56.4154) (width 0.3) (layer F.Cu) (net 45))
   (segment (start 147.022 63.0682) (end 147.022 61.848) (width 0.3) (layer F.Cu) (net 45))
   (via (at 151.75 69.16) (size 0.6) (drill 0.3) (layers F.Cu B.Cu) (net 45))
   (segment (start 151.6444 69.2656) (end 151.75 69.16) (width 0.3) (layer F.Cu) (net 45))
   (segment (start 151.6444 71.7976) (end 151.6444 69.2656) (width 0.3) (layer F.Cu) (net 45))
-  (segment (start 147.59 61.57) (end 147.445 61.425) (width 0.3) (layer F.Cu) (net 45))
-  (segment (start 147.022 61.848) (end 147.27 61.6) (width 0.3) (layer F.Cu) (net 45))
-  (segment (start 147.27 61.6) (end 147.445 61.425) (width 0.3) (layer F.Cu) (net 45))
-  (segment (start 147.56 61.31) (end 147.6 61.27) (width 0.3) (layer F.Cu) (net 45))
-  (segment (start 147.445 61.425) (end 147.6 61.27) (width 0.3) (layer F.Cu) (net 45))
-  (segment (start 147.71 61.69) (end 147.71 61.16) (width 0.3) (layer F.Cu) (net 45))
-  (segment (start 147.73 61.14) (end 147.89 60.98) (width 0.3) (layer F.Cu) (net 45))
-  (segment (start 147.71 61.16) (end 147.73 61.14) (width 0.3) (layer F.Cu) (net 45))
-  (segment (start 147.71 61.69) (end 147.59 61.57) (width 0.3) (layer F.Cu) (net 45))
-  (segment (start 147.6 61.27) (end 147.73 61.14) (width 0.3) (layer F.Cu) (net 45))
-  (segment (start 147.62 61.6) (end 147.71 61.69) (width 0.3) (layer F.Cu) (net 45))
-  (segment (start 147.27 61.6) (end 147.62 61.6) (width 0.3) (layer F.Cu) (net 45))
   (segment (start 151.75 64.28) (end 151.75 63.43) (width 0.3) (layer B.Cu) (net 45))
   (segment (start 151.75 63.792167) (end 151.75 64.28) (width 0.3) (layer B.Cu) (net 45))
@@
   (segment (start 151.75 63.43) (end 151.74 63.42) (width 0.3) (layer B.Cu) (net 45))
   (segment (start 151.75 64.28) (end 151.75 69.16) (width 0.3) (layer B.Cu) (net 45))
-  (segment (start 151.244951 62.500687) (end 148.520687 62.500687) (width 0.3) (layer F.Cu) (net 45))
-  (segment (start 148.520687 62.500687) (end 147.71 61.69) (width 0.3) (layer F.Cu) (net 45))
-  (segment (start 151.74 62.995736) (end 151.244951 62.500687) (width 0.3) (layer F.Cu) (net 45))
   (segment (start 151.74 63.42) (end 151.74 62.995736) (width 0.3) (layer F.Cu) (net 45))
+  (segment (start 147.022 60.222256) (end 147.022 62.6682) (width 0.3) (layer F.Cu) (net 45))
+  (segment (start 147.022 62.6682) (end 147.022 63.0682) (width 0.3) (layer F.Cu) (net 45))
+  (segment (start 147.732128 59.512128) (end 147.74501 59.499246) (width 0.3) (layer F.Cu) (net 45))
+  (segment (start 147.74501 59.499246) (end 147.760754 59.499246) (width 0.3) (layer F.Cu) (net 45))
+  (segment (start 147.732128 59.512128) (end 147.022 60.222256) (width 0.3) (layer F.Cu) (net 45))
+  (segment (start 150.8446 56.4154) (end 151.877 56.4154) (width 0.3) (layer F.Cu) (net 45))
+  (segment (start 147.760754 59.499246) (end 150.8446 56.4154) (width 0.3) (layer F.Cu) (net 45))
+  (segment (start 151.74 56.5524) (end 151.877 56.4154) (width 0.3) (layer F.Cu) (net 45))
+  (segment (start 151.74 63.42) (end 151.74 56.5524) (width 0.3) (layer F.Cu) (net 45))
   (via (at 150.79926 69.194536) (size 0.6) (drill 0.3) (layers F.Cu B.Cu) (net 46))
   (segment (start 150.8444 69.239676) (end 150.79926 69.194536) (width 0.3) (layer F.Cu) (net 46))

Commit message: fix logos
Parts:
- moved REF** 4.48 mm to (138.9, 59.6)
- moved G*** 4.01 mm to (139.4, 67.8)
- moved R5 2.44 mm to (156.5, 66.9), turned to 270 degrees
- moved D1 1.64 mm to (133.6, 56.7)
- moved R4 1.21 mm to (143.1, 70.4)
Routing:
- net GND: track 102.9 -> 116.0 mm, vias 12 -> 15
- net +3V3: track 141.6 -> 146.7 mm, vias 3 -> 5
- net Net-(D5-Pad1): track 5.23 -> 8.44 mm
- net Net-(D1-Pad1): track 4.51 -> 2.85 mm
- net Net-(D4-Pad1): track 5.08 -> 6.24 mm

Commit message: logos ok, and labels
Parts:
- moved G*** 8.97 mm to (139.2, 76.8)
- moved REF** 2.19 mm to (139.3, 61.8)
- moved G*** 1.89 mm to (141.2, 79.7)
- renumbered D3 to CHG, D4 to LED1, D5 to LED2, D6 to LED3, SW2 to MAGSPOOF, SW3 to NFC, D1 to PWR, SW1 to RESET
Other:
- board text added: "Battery"
- board text removed: "battery"
Changed lines of the file:
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@@
-(kicad_pcb (version 20171130) (host pcbnew "(5.1.4-0-10_14)")
+(kicad_pcb (version 20171130) (host pcbnew "(5.1.5-0-10_14)")
   (general
     (thickness 1.6)
@@
   )
   (page A4)
+  (title_block
+    (title "NFC Copy Cat")
+    (date 2020-02-10)
+    (rev 1.3)
+    (company "Electronic Cats")
+    (comment 3 "Andres Sabas")
+    (comment 4 "Montserrat Figueroa")
+  )
   (layers
     (0 F.Cu signal)
@@
     (tags "SPST Tactile Switch")
     (attr smd)
-    (fp_text reference SW2 (at -0.01 -3.82) (layer B.SilkS)
+    (fp_text reference MAGSPOOF (at -0.01 -3.82) (layer B.SilkS)
       (effects (font (size 1 1) (thickness 0.15)) (justify mirror))
     )
@@
     (descr "Through hole straight pin header, 1x08, 2.54mm pitch, single row")
     (tags "Through hole pin header THT 1x08 2.54mm single row")
-    (fp_text reference J4 (at 0.12 19.86 90) (layer F.SilkS)
+    (fp_text reference J4 (at 0.17 20.45 90) (layer F.SilkS)
       (effects (font (size 1 1) (thickness 0.15)))
     )
@@
     (tags "SPST Tactile Switch")
     (attr smd)
-    (fp_text reference SW3 (at -0.1 -3.65 180) (layer B.SilkS)
+    (fp_text reference NFC (at -0.1 -3.65 180) (layer B.SilkS)
       (effects (font (size 1 1) (thickness 0.15)) (justify mirror))
     )
@@
   )
   (module Aesthetics:electronic_cats_logo_8x6 (layer B.Cu)
-    (at 139.36 67.79 180)
+    (at 139.18 76.76 180)
     (fp_text reference G*** (at 0 0) (layer B.SilkS) hide
       (effects (font (size 1.524 1.524) (thickness 0.3)) (justify mirror))
@@
   )
   (module Symbol:OSHW-Logo2_7.3x6mm_SilkScreen (layer B.Cu)
-    (at 138.86 59.64 180)
+    (at 139.35 61.77 180)
     (descr "Open Source Hardware Symbol")
     (tags "Logo Symbol OSHW")
@@
   )
   (module Aesthetics:electronic_cats_logo_4x3 (layer F.Cu)
-    (at 139.5095 78.8035)
+    (at 141.17 79.71)
     (fp_text reference G*** (at 0 0) (layer F.SilkS) hide
       (effects (font (size 1.524 1.524) (thickness 0.3)))
@@
     (tags "SOIC SO")
     (attr smd)
-    (fp_text reference U3 (at 2.575 -4.245) (layer F.SilkS)
+    (fp_text reference U3 (at 1.925 -3.415) (layer F.SilkS)
       (effects (font (size 1 1) (thickness 0.15)))
     )
@@
     (tags "LED handsolder")
     (attr smd)
-    (fp_text reference D1 (at 2.825 -0.03) (layer F.SilkS)
+    (fp_text reference PWR (at 3.685 -0.12) (layer F.SilkS)
       (effects (font (size 1 1) (thickness 0.15)))
     )
@@
     (tags "LED handsolder")
     (attr smd)
-    (fp_text reference D3 (at 3.405 -0.09) (layer F.SilkS)
+    (fp_text reference CHG (at 3.405 -0.09) (layer F.SilkS)
       (effects (font (size 1 1) (thickness 0.15)))
     )
@@
     (descr "Through hole straight pin header, 1x02, 2.54mm pitch, single row")
     (tags "Through hole pin header THT 1x02 2.54mm single row")
-    (fp_text reference J2 (at -1.205 -2.025 180) (layer F.SilkS)
+    (fp_text reference J2 (at 0.074 -2.4592 180) (layer F.SilkS)
       (effects (font (size 1 1) (thickness 0.15)))
     )
@@
     (descr "Through hole straight pin header, 1x02, 2.54mm pitch, single row")
     (tags "Through hole pin header THT 1x02 2.54mm single row")
-    (fp_text reference J5 (at -0.12 -2.37 180) (layer F.SilkS)
-      (effects (font (size 1 1) (thickness 0.15)))
+    (fp_text reference J5 (at -0.12 -2.37 -180) (layer B.SilkS)
+      (effects (font (size 1 1) (thickness 0.15)) (justify mirror))
     )
     (fp_text value Conn_01x02 (at 0 4.87) (layer F.Fab)
@@
     (tags "SPST Tactile Switch")
     (attr smd)
-    (fp_text reference SW1 (at -0.03 -3.64) (layer B.SilkS)
+    (fp_text reference RESET (at -0.03 -3.64) (layer B.SilkS)
       (effects (font (size 1 1) (thickness 0.15)) (justify mirror))
     )
@@
     (tags "LED handsolder")
     (attr smd)
-    (fp_text reference D4 (at 3.115 -0.11 90) (layer B.SilkS)
+    (fp_text reference LED1 (at 0.145 1.68 90) (layer B.SilkS)
       (effects (font (size 1 1) (thickness 0.15)) (justify mirror))
     )
@@
     (tags "LED handsolder")
     (attr smd)
-    (fp_text reference D5 (at 2.885 0.01 90) (layer B.SilkS)
+    (fp_text reference LED2 (at 3.655 -0.02 90) (layer B.SilkS)
       (effects (font (size 1 1) (thickness 0.15)) (justify mirror))
     )
@@
     (tags "LED handsolder")
     (attr smd)
-    (fp_text reference D6 (at 3.005 0.07 90) (layer B.SilkS)
+    (fp_text reference LED3 (at 3.775 -0.07 90) (layer B.SilkS)
       (effects (font (size 1 1) (thickness 0.15)) (justify mirror))
     )
@@
     (descr "Through hole straight pin header, 1x09, 2.54mm pitch, single row")
     (tags "Through hole pin header THT 1x09 2.54mm single row")
-    (fp_text reference J6 (at 0 -2.33) (layer F.SilkS)
+    (fp_text reference J6 (at -0.72 -2.64) (layer F.SilkS)
       (effects (font (size 1 1) (thickness 0.15)))
     )
@@
     (effects (font (size 1 1) (thickness 0.15)))
   )
-  (gr_text battery (at 130.25 87.01) (layer B.SilkS)
-    (effects (font (size 1 1) (thickness 0.15)) (justify mirror))
+  (gr_text Battery (at 132.07 87.76) (layer F.SilkS)
+    (effects (font (size 1 1) (thickness 0.15)))
   )
   (gr_text + (at 138.4052 81.1412 90) (layer F.SilkS)
@@
     (effects (font (size 1 1) (thickness 0.15)))
   )
-  (gr_text "NFC COPY CAT \nv1.3" (at 134.77 52.53) (layer B.SilkS)
+  (gr_text "NFC COPY CAT \nv1.3" (at 136.38 70.17) (layer B.SilkS)
     (effects (font (size 1 1) (thickness 0.15)) (justify mirror))
   )

Commit message: fix pin
Parts:
- moved J4 17.8 mm to (162.2, 64.8), turned to 0 degrees
- moved G*** 8.97 mm to (139.4, 67.8)
- moved REF** 2.19 mm to (138.9, 59.6)
- moved G*** 1.89 mm to (139.5, 78.8)
- renumbered PWR to D1, CHG to D3, LED1 to D4, LED2 to D5, LED3 to D6, RESET to SW1, MAGSPOOF to SW2, NFC to SW3
Routing:
- net /IRQ: track 30.9 -> 12.8 mm, vias 1 -> 0
- net /12(MISO): track 37.9 -> 44.1 mm, vias 1 -> 3
- net GND: track 116.0 -> 122.2 mm, vias 15 -> 14
- net /13(SCK): track 56.4 -> 59.4 mm
- net +3V3: track 146.7 -> 149.4 mm
- net /11(MOSI): track 40.6 -> 38.0 mm, vias 2 -> 1
- net /IN_B: track 26.4 -> 25.5 mm
- net /10(SS): track 37.8 -> 38.5 mm, vias 2 -> 1
Other:
- board text added: "battery"
- board text removed: "Battery"
