File: hardware/nfc_copy_cat.kicad_pcb (KiCad board)
At the start: 2 copper layers, 40.4 x 43 mm, 41 parts, among them J1 USB_B_Micro, J2 Battery, J3 SWD, J4 NFC Module V3, J5 Conn_01x02, J6 Adafruit NFC 1.0, SW1 RST, SW2 Magspoof, SW3 NFC, U1 AP2112K-3.3TRG1, U2 MCP73831-2-OT, U3 TC4424, U4 ATSAMD21E18A, U5 W25Q16JVSS

Commit message: chance labels
Routing:
- net /13(SCK): track 59.4 -> 57.2 mm
Changed lines of the file:
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@@
     (thickness 1.6)
     (drawings 32)
-    (tracks 629)
+    (tracks 622)
     (zones 0)
     (modules 41)
@@
     (descr "Through hole straight pin header, 1x08, 2.54mm pitch, single row")
     (tags "Through hole pin header THT 1x08 2.54mm single row")
-    (fp_text reference J4 (at 0.12 19.86 90) (layer F.SilkS)
+    (fp_text reference J4 (at -0.21 -2.44 180) (layer F.SilkS)
       (effects (font (size 1 1) (thickness 0.15)))
     )
-    (fp_text value "NFC Module V3" (at 0 20.11) (layer F.Fab)
+    (fp_text value "NFC Module V3" (at -0.37 20.2) (layer F.Fab)
       (effects (font (size 1 1) (thickness 0.15)))
     )
@@
     (descr U254-051N-4BH806-2)
     (tags Connector)
-    (fp_text reference J1 (at -4.7975 2.8015 -180) (layer F.SilkS)
+    (fp_text reference J1 (at -4.7975 2.8015 -180) (layer F.Fab)
       (effects (font (size 1 1) (thickness 0.15)))
     )
@@
     (tags "SOIC SO")
     (attr smd)
-    (fp_text reference U3 (at 2.575 -4.245) (layer F.SilkS)
+    (fp_text reference U3 (at 2.085 -3.375) (layer F.SilkS)
       (effects (font (size 1 1) (thickness 0.15)))
     )
@@
     (descr "Through hole straight pin header, 1x02, 2.54mm pitch, single row")
     (tags "Through hole pin header THT 1x02 2.54mm single row")
-    (fp_text reference J2 (at -1.205 -2.025 180) (layer F.SilkS)
+    (fp_text reference J2 (at -2.556 1.0908 180) (layer F.SilkS)
       (effects (font (size 1 1) (thickness 0.15)))
     )
@@
     (descr "Through hole straight pin header, 1x02, 2.54mm pitch, single row")
     (tags "Through hole pin header THT 1x02 2.54mm single row")
-    (fp_text reference J5 (at -0.12 -2.37 180) (layer F.SilkS)
+    (fp_text reference J5 (at 2.7 0 90) (layer F.SilkS)
       (effects (font (size 1 1) (thickness 0.15)))
     )
@@
     (descr "Through hole straight pin header, 1x09, 2.54mm pitch, single row")
     (tags "Through hole pin header THT 1x09 2.54mm single row")
-    (fp_text reference J6 (at 0 -2.33) (layer F.SilkS)
+    (fp_text reference J6 (at -0.17 -2.52) (layer F.SilkS)
       (effects (font (size 1 1) (thickness 0.15)))
     )
@@
     (effects (font (size 1 1) (thickness 0.15)))
   )
-  (gr_text Coil (at 166.57 88.95 90) (layer F.SilkS)
+  (gr_text Coil (at 166.56 90.05 90) (layer F.SilkS)
     (effects (font (size 1 1) (thickness 0.15)))
   )
-  (gr_text battery (at 130.25 87.01) (layer B.SilkS)
+  (gr_text battery (at 130.76 87.52) (layer B.SilkS)
     (effects (font (size 1 1) (thickness 0.15)) (justify mirror))
   )
@@
     (effects (font (size 0.7 0.7) (thickness 0.15)) (justify mirror))
   )
-  (gr_text SCK (at 159.21 82.77) (layer F.SilkS)
+  (gr_text SCK (at 159.34 65.09) (layer F.SilkS)
     (effects (font (size 1 1) (thickness 0.15)))
   )
-  (gr_text MISO (at 158.81 80.18) (layer F.SilkS)
+  (gr_text MISO (at 158.97 67.43) (layer F.SilkS)
     (effects (font (size 1 1) (thickness 0.15)))
   )
-  (gr_text MOSI (at 158.92 77.59) (layer F.SilkS)
+  (gr_text MOSI (at 158.93 69.86) (layer F.SilkS)
     (effects (font (size 1 1) (thickness 0.15)))
   )
-  (gr_text SS (at 159.46 74.98) (layer F.SilkS)
+  (gr_text SS (at 159.54 72.41) (layer F.SilkS)
     (effects (font (size 1 1) (thickness 0.15)))
   )
-  (gr_text 3V3 (at 159.3 72.65) (layer F.SilkS)
+  (gr_text 3V3 (at 159.3 74.83) (layer F.SilkS)
     (effects (font (size 1 1) (thickness 0.15)))
   )
-  (gr_text GND (at 159.22 69.88) (layer F.SilkS)
+  (gr_text GND (at 159.13 77.46) (layer F.SilkS)
     (effects (font (size 1 1) (thickness 0.15)))
   )
-  (gr_text IRQ (at 159.4 67.46) (layer F.SilkS)
+  (gr_text IRQ (at 159.17 80.22) (layer F.SilkS)
     (effects (font (size 1 1) (thickness 0.15)))
   )
@@
   (segment (start 160.67 61.07) (end 160.67 66.576436) (width 0.5) (layer B.Cu) (net 1))
   (segment (start 157.7076 71.7976) (end 159.3576 71.7976) (width 0.5) (layer F.Cu) (net 1))
-  (segment (start 162.17 74.99) (end 160.76 73.58) (width 0.5) (layer F.Cu) (net 1))
-  (segment (start 160.76 73.58) (end 160.76 70.85) (width 0.5) (layer F.Cu) (net 1))
-  (segment (start 160.76 70.85) (end 160.346504 70.436504) (width 0.5) (layer F.Cu) (net 1))
   (segment (start 159.536504 70.139512) (end 159.833496 70.436504) (width 0.5) (layer F.Cu) (net 1))
   (segment (start 159.536504 70.436504) (end 159.536504 70.033496) (width 0.5) (layer F.Cu) (net 1))
   (segment (start 159.833496 70.436504) (end 159.536504 70.436504) (width 0.5) (layer F.Cu) (net 1))
-  (segment (start 160.346504 70.436504) (end 159.833496 70.436504) (width 0.5) (layer F.Cu) (net 1))
   (segment (start 159.536504 70.033496) (end 159.536504 70.139512) (width 0.5) (layer F.Cu) (net 1))
   (segment (start 159.536504 70.733496) (end 159.833496 70.436504) (width 0.5) (layer F.Cu) (net 1))
@@
   (segment (start 159.536504 71.016504) (end 159.536504 70.436504) (width 0.5) (layer F.Cu) (net 1))
   (segment (start 159.536504 70.033496) (end 159.536504 68.46552) (width 0.5) (layer F.Cu) (net 1))
+  (segment (start 162.17 74.99) (end 160.76 73.58) (width 0.5) (layer F.Cu) (net 1))
+  (segment (start 160.346504 70.436504) (end 159.833496 70.436504) (width 0.5) (layer F.Cu) (net 1))
+  (segment (start 160.76 70.85) (end 160.346504 70.436504) (width 0.5) (layer F.Cu) (net 1))
+  (segment (start 160.76 73.58) (end 160.76 70.85) (width 0.5) (layer F.Cu) (net 1))
   (via (at 132.334 78.486) (size 0.6) (drill 0.3) (layers F.Cu B.Cu) (net 2))
   (segment (start 133.83 78.47) (end 132.35 78.47) (width 0.3) (layer F.Cu) (net 2))
@@
   (segment (start 152.5775 90.7475) (end 151.13 89.3) (width 0.3) (layer F.Cu) (net 2))
   (segment (start 151.13 86.21) (end 151.13 87.77) (width 0.3) (layer F.Cu) (net 2))
-  (via (at 131.04 64.31) (size 0.6) (drill 0.3) (layers F.Cu B.Cu) (net 2))
-  (segment (start 133.2296 64.31) (end 131.04 64.31) (width 0.3) (layer F.Cu) (net 2))
-  (segment (start 133.5532 64.6336) (end 133.2296 64.31) (width 0.3) (layer F.Cu) (net 2))
-  (segment (start 133.5532 65.7136) (end 133.5532 64.6336) (width 0.3) (layer F.Cu) (net 2))
   (via (at 157.25 85.72) (size 0.6) (drill 0.3) (layers F.Cu B.Cu) (net 2))
   (via (at 141.66 56.73) (size 0.6) (drill 0.3) (layers F.Cu B.Cu) (net 2))
@@
   (segment (start 163.990011 80.330011) (end 163.420001 79.760001) (width 0.3) (layer B.Cu) (net 2))
   (segment (start 164.120011 80.330011) (end 163.990011 80.330011) (width 0.3) (layer B.Cu) (net 2))
+  (segment (start 133.5532 65.7136) (end 133.5532 64.6336) (width 0.3) (layer F.Cu) (net 2))
+  (segment (start 133.5532 64.6336) (end 133.2296 64.31) (width 0.3) (layer F.Cu) (net 2))
+  (segment (start 133.2296 64.31) (end 131.04 64.31) (width 0.3) (layer F.Cu) (net 2))
+  (via (at 131.04 64.31) (size 0.6) (drill 0.3) (layers F.Cu B.Cu) (net 2))
   (segment (start 138.845 73.31) (end 138.8285 73.2935) (width 0.5) (layer F.Cu) (net 3))
   (segment (start 143.13 73.31) (end 138.845 73.31) (width 0.5) (layer F.Cu) (net 3))
@@
   (segment (start 144.88 81.12) (end 144.88 81.29) (width 0.3) (layer B.Cu) (net 13))
   (segment (start 160.847965 84.028001) (end 160.504986 83.685022) (width 0.3) (layer F.Cu) (net 13))
-  (segment (start 162.05 83.76) (end 162.06 83.76) (width 0.3) (layer F.Cu) (net 13))
   (via (at 160.204987 83.385023) (size 0.6) (drill 0.3) (layers F.Cu B.Cu) (net 13))
-  (segment (start 162.05 83.76) (end 162.041999 83.768001) (width 0.3) (layer F.Cu) (net 13))
-  (segment (start 162.041999 83.768001) (end 162.041999 84.028001) (width 0.3) (layer F.Cu) (net 13))
   (segment (start 162.041999 84.028001) (end 162.328001 84.028001) (width 0.3) (layer F.Cu) (net 13))
-  (segment (start 161.878001 83.931999) (end 162.05 83.76) (width 0.3) (layer F.Cu) (net 13))
-  (segment (start 161.878001 84.028001) (end 161.878001 83.931999) (width 0.3) (layer F.Cu) (net 13))
   (segment (start 161.878001 84.028001) (end 160.847965 84.028001) (width 0.3) (layer F.Cu) (net 13))
-  (segment (start 162.05 82.61) (end 162.05 83.76) (width 0.3) (layer F.Cu) (net 13))
   (segment (start 160.504986 83.685022) (end 160.204987 83.385023) (width 0.3) (layer F.Cu) (net 13))
   (segment (start 161.878001 84.028001) (end 162.041999 84.028001) (width 0.3) (layer F.Cu) (net 13))
-  (segment (start 162.06 83.76) (end 162.328001 84.028001) (width 0.3) (layer F.Cu) (net 13))
   (segment (start 165.83 64.83) (end 165.84 64.82) (width 0.3) (layer F.Cu) (net 13))
   (segment (start 162.17 64.83) (end 165.83 64.83) (width 0.3) (layer F.Cu) (net 13))
